File: Voyager104.kicad_pcb (KiCad board)
At the start: 2 copper layers, 343.7 x 123.4 mm, 308 parts, among them J1 AVR-ISP-6, Q1 DSS60601MZ4-13, SW1 SW_Push, U1 AT90USB1286-AU, U2 PRTR5V0U2X, Y1 16MHz

Commit message: Build PCB
Parts:
- added D102: SOD-323, Diodes_SMD:D_SOD-123, B.Cu at (446.1, 92.1)
- added D103: SOD-323, Diodes_SMD:D_SOD-123, B.Cu at (408.0, 119.1)
- added D104: SOD-323, Diodes_SMD:D_SOD-123, B.Cu at (427.0, 119.1)
- added D105: SOD-323, Diodes_SMD:D_SOD-123, B.Cu at (430.2, 119.1)
- added D106: SOD-323, Diodes_SMD:D_SOD-123, B.Cu at (449.3, 111.1)
- added D107: SOD-323, Diodes_SMD:D_SOD-123, B.Cu at (392.1, 138.1)
- added D109: SOD-323, Diodes_SMD:D_SOD-123, B.Cu at (427.0, 138.1)
- added D110: SOD-323, Diodes_SMD:D_SOD-123, B.Cu at (430.2, 138.1)
- added D114: SOD-323, Diodes_SMD:D_SOD-123, B.Cu at (446.1, 130.2)
- added D15: SOD-323, Diodes_SMD:D_SOD-123, B.Cu at (408.0, 38.1)
- added D16: SOD-323, Diodes_SMD:D_SOD-123, B.Cu at (427.0, 38.1)
- added D32: SOD-323, Diodes_SMD:D_SOD-123, B.Cu at (446.1, 38.1)
- added D33: SOD-323, Diodes_SMD:D_SOD-123, B.Cu at (449.3, 38.1)
- added D34: SOD-323, Diodes_SMD:D_SOD-123, B.Cu at (408.0, 61.9)
- added D49: SOD-323, Diodes_SMD:D_SOD-123, B.Cu at (427.0, 61.9)
- added D50: SOD-323, Diodes_SMD:D_SOD-123, B.Cu at (446.1, 61.9)
- added D51: SOD-323, Diodes_SMD:D_SOD-123, B.Cu at (449.3, 61.9)
- added D64: SOD-323, Diodes_SMD:D_SOD-123, B.Cu at (408.0, 81.0)
- added D79: SOD-323, Diodes_SMD:D_SOD-123, B.Cu at (427.0, 81.0)
- added D80: SOD-323, Diodes_SMD:D_SOD-123, B.Cu at (430.2, 81.0)
- added D83: SOD-323, Diodes_SMD:D_SOD-123, B.Cu at (449.3, 73.0)
- added D88: SOD-323, Diodes_SMD:D_SOD-123, B.Cu at (408.0, 100.0)
- added D89: SOD-323, Diodes_SMD:D_SOD-123, B.Cu at (427.0, 100.0)
- added D98: SOD-323, Diodes_SMD:D_SOD-123, B.Cu at (430.2, 100.0)
- added MX_NUM1: MX-1U, MX_Alps_Hybrid:MX-1U, F.Cu at (400.1, 39.7)
- added MX_NUM10: MX-1U, MX_Alps_Hybrid:MX-1U, F.Cu at (419.1, 82.5)
- added MX_NUM11: MX-1U, MX_Alps_Hybrid:MX-1U, F.Cu at (438.1, 82.5)
- added MX_NUM12: MX-1U, MX_Alps_Hybrid:MX-1U, F.Cu at (457.2, 82.5)
- added MX_NUM13: MX-1U, MX_Alps_Hybrid:MX-1U, F.Cu at (400.1, 101.6)
- added MX_NUM14: MX-1U, MX_Alps_Hybrid:MX-1U, F.Cu at (419.1, 101.6)
- added MX_NUM15: MX-1U, MX_Alps_Hybrid:MX-1U, F.Cu at (438.1, 101.6)
- added MX_NUM16: MX-1U, MX_Alps_Hybrid:MX-1U, F.Cu at (457.2, 101.6)
- added MX_NUM17: MX-1U, MX_Alps_Hybrid:MX-1U, F.Cu at (400.1, 120.7)
- added MX_NUM18: MX-1U, MX_Alps_Hybrid:MX-1U, F.Cu at (419.1, 120.7)
- added MX_NUM19: MX-1U, MX_Alps_Hybrid:MX-1U, F.Cu at (438.1, 120.7)
- added MX_NUM2: MX-1U, MX_Alps_Hybrid:MX-1U, F.Cu at (419.1, 39.7)
- added MX_NUM20: MX-1U, MX_Alps_Hybrid:MX-1U, F.Cu at (457.2, 120.7)
- added MX_NUM21: MX-1U, MX_Alps_Hybrid:MX-1U, F.Cu at (400.1, 139.7)
- added MX_NUM22: MX-1U, MX_Alps_Hybrid:MX-1U, F.Cu at (419.1, 139.7)
- added MX_NUM23: MX-1U, MX_Alps_Hybrid:MX-1U, F.Cu at (438.1, 139.7)
- added MX_NUM24: MX-1U, MX_Alps_Hybrid:MX-1U, F.Cu at (457.2, 139.7)
- added MX_NUM3: MX-1U, MX_Alps_Hybrid:MX-1U, F.Cu at (438.1, 39.7)
- added MX_NUM4: MX-1U, MX_Alps_Hybrid:MX-1U, F.Cu at (457.2, 39.7)
- added MX_NUM5: MX-1U, MX_Alps_Hybrid:MX-1U, F.Cu at (400.1, 63.5)
- added MX_NUM6: MX-1U, MX_Alps_Hybrid:MX-1U, F.Cu at (419.1, 63.5)
- added MX_NUM7: MX-1U, MX_Alps_Hybrid:MX-1U, F.Cu at (438.1, 63.5)
- added MX_NUM8: MX-1U, MX_Alps_Hybrid:MX-1U, F.Cu at (457.2, 63.5)
- added MX_NUM9: MX-1U, MX_Alps_Hybrid:MX-1U, F.Cu at (400.1, 82.5)
- added MX_NUM_EX1: MX-2U, MX_Alps_Hybrid:MX-2U-ReversedStabilizers, F.Cu at (457.2, 92.1)
- added MX_NUM_EX2: MX-2U, MX_Alps_Hybrid:MX-2U-ReversedStabilizers, F.Cu at (457.2, 130.2)
- added MX_NUM_EX3: MX-2U, MX_Alps_Hybrid:MX-2U-ReversedStabilizers, F.Cu at (409.6, 139.7)
- added R102: 1k, Resistors_SMD:R_0603, B.Cu at (446.1, 97.6)
- added R103: 1k, Resistors_SMD:R_0603, B.Cu at (408.0, 124.6)
- added R104: 1k, Resistors_SMD:R_0603, B.Cu at (427.0, 124.6)
- added R105: 1k, Resistors_SMD:R_0603, B.Cu at (430.2, 124.6)
- added R106: 1k, Resistors_SMD:R_0603, B.Cu at (449.3, 123.0)
- added R107: 1k, Resistors_SMD:R_0603, B.Cu at (392.1, 143.7)
- added R109: 1k, Resistors_SMD:R_0603, B.Cu at (427.0, 143.7)
- added R110: 1k, Resistors_SMD:R_0603, B.Cu at (430.2, 143.7)
- added R114: 1k, Resistors_SMD:R_0603, B.Cu at (446.1, 135.7)
- added R15: 1k, Resistors_SMD:R_0603, B.Cu at (408.0, 43.7)
- added R34: 1k, Resistors_SMD:R_0603, B.Cu at (427.0, 43.7)
- added R49: 1k, Resistors_SMD:R_0603, B.Cu at (446.1, 43.7)
- added R50: 1k, Resistors_SMD:R_0603, B.Cu at (449.3, 43.7)
- added R51: 1k, Resistors_SMD:R_0603, B.Cu at (408.0, 67.5)
- added R64: 1k, Resistors_SMD:R_0603, B.Cu at (427.0, 67.5)
- added R79: 1k, Resistors_SMD:R_0603, B.Cu at (446.1, 67.5)
- added R80: 1k, Resistors_SMD:R_0603, B.Cu at (449.3, 67.5)
- added R83: 1k, Resistors_SMD:R_0603, B.Cu at (408.0, 86.5)
- added R88: 1k, Resistors_SMD:R_0603, B.Cu at (427.0, 86.5)
- added R89: 1k, Resistors_SMD:R_0603, B.Cu at (430.2, 86.5)
- added R92: 1k, Resistors_SMD:R_0603, B.Cu at (449.3, 84.9)
- added R93: 1k, Resistors_SMD:R_0603, B.Cu at (408.0, 105.6)
- added R94: 1k, Resistors_SMD:R_0603, B.Cu at (427.0, 105.6)
- added R98: 1k, Resistors_SMD:R_0603, B.Cu at (430.2, 105.6)
- moved G*** 223.8 mm to (357.2, 51.6) (x2)
- moved G*** 148.7 mm to (376.2, 120.7)
- moved D101 15.9 mm to (384.2, 81.0)
- moved D113 15.9 mm to (384.2, 138.1)
- moved D94 15.9 mm to (384.2, 38.1)
- moved D97 15.9 mm to (384.2, 61.9)
- moved R101 15.9 mm to (384.2, 86.5)
- moved R113 15.9 mm to (384.2, 143.7)
- moved R33 15.9 mm to (384.2, 43.7)
- moved R97 15.9 mm to (384.2, 67.5)
Connections:
- U1 pad 33: Net-(U1-Pad33) -> COL20
- U1 pad 34: Net-(U1-Pad34) -> COL19
- U1 pad 35: Net-(U1-Pad35) -> COL18
- U1 pad 36: Net-(U1-Pad36) -> COL17
Routing:
- net +5V: track 2378.9 -> 2935.1 mm
- net LEDGND: track 1796.0 -> 2285.2 mm, vias 17 -> 18
- net COL20: track 0.00 -> 216.3 mm, vias 0 -> 1
- net COL19: track 0.00 -> 195.1 mm, vias 0 -> 1
- net COL18: track 0.00 -> 178.0 mm
- net COL17: track 0.00 -> 171.2 mm
- net ROW3: track 367.0 -> 487.5 mm, vias 4 -> 5
- net ROW4: track 322.8 -> 419.6 mm
- net ROW2: track 423.4 -> 519.3 mm
- net ROW5: track 359.6 -> 449.7 mm
- net ROW1: track 448.9 -> 539.0 mm
- net ROW0: track 464.7 -> 554.6 mm
- net Net-(MX_NUM24-Pad4): track 0.00 -> 34.5 mm
- net Net-(MX_NUM16-Pad4): track 0.00 -> 34.5 mm
- net Net-(D107-Pad2): track 0.00 -> 24.3 mm
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Other:
- board size 343.7 x 123.4 mm -> 425.4 x 123.4 mm
- board text added: "104"
- board text added: "Voyager104 PCB Rev 1.0 20190216"
- board text removed: "87"
- board text removed: "Voyager87 PCB Rev 1.0 20190211"
