File: Voyager104.sch (KiCad schematic (older format))
At the start: 22 parts, among them J1 AVR-ISP-6, Q1 DSS60601MZ4-13, SW1 SW_Push, U1 AT90USB1286-AU, U2 PRTR5V0U2X, Y1 16MHz

Commit message: Build PCB
Connections:
- net labels added: COL17, COL18, COL19, COL20
Changed lines of the file:
@@
 EESchema Schematic File Version 4
-LIBS:Voyager87-cache
+LIBS:Voyager104-cache
 EELAYER 26 0
 EELAYER END
@@
 Connection ~ 4000 2975
 Connection ~ 3725 3275
+Text GLabel 5125 5175 2    50   Input ~ 0
+COL17
+Text GLabel 5125 5075 2    50   Input ~ 0
+COL18
+Text GLabel 3925 5175 0    50   Input ~ 0
+COL19
+Text GLabel 3925 5075 0    50   Input ~ 0
+COL20
 $EndSCHEMATC
