File: matrix.sch (KiCad schematic (older format))
At the start: 283 parts

Commit message: Build PCB
Parts:
- added D102, D103, D104, D105, D106, D107, D109, D110, D114, D15, D16, D32, D33, D34, D49, D50, D51, D64, D79, D80, D83, D88, D89, D98: SOD-323, Diodes_SMD:D_SOD-123, symbol Device:D_Small
- added MX_NUM1, MX_NUM10, MX_NUM11, MX_NUM12, MX_NUM13, MX_NUM14, MX_NUM15, MX_NUM16, MX_NUM17, MX_NUM18, MX_NUM19, MX_NUM2, MX_NUM20, MX_NUM21, MX_NUM22, MX_NUM23, MX_NUM24, MX_NUM3, MX_NUM4, MX_NUM5, MX_NUM6, MX_NUM7, MX_NUM8, MX_NUM9: MX-1U, MX_Alps_Hybrid:MX-1U, symbol MX_Alps_Hybrids:MX-1U
- added MX_NUM_EX1, MX_NUM_EX2, MX_NUM_EX3: MX-2U, MX_Alps_Hybrid:MX-2U-ReversedStabilizers, symbol MX_Alps_Hybrids:MX-1U
- added R102, R103, R104, R105, R106, R107, R109, R110, R114, R15, R34, R49, R50, R51, R64, R79, R80, R83, R88, R89, R92, R93, R94, R98: 1k, Resistors_SMD:R_0603, symbol Device:R_Small
Connections:
- net labels added: COL17, COL18, COL19, COL20
- wire segments 909 -> 1142
